File: bmx280-i2c-adapter.kicad/bmx280-i2c-adapter.kicad_pcb (KiCad board)
At the start: 2 copper layers, 20 x 34 mm, 13 parts, among them J1 Stemma-QT_Qwicc, J2 Stemma-QT_Qwicc, J3 Stemma-QT_Qwicc, J4 Stemma-QT_Qwicc, J5 Grove, J6 Grove, U1 BMx280

Commit message: Rev 1.01: add assembly for Stemma/Qt on top side
Other:
- board text added: "Rev: 1.01"
- board text removed: "Rev: 1.00"
Changed lines of the file:
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@@
     (descr "JST SH series connector, SM04B-SRSS-TB (http://www.jst-mfg.com/product/pdf/eng/eSH.pdf), generated with kicad-footprint-generator")
     (tags "connector JST SH top entry")
-    (property "LCSC" "")
-    (property "Sheetfile" "bmx280-i2c-adapter.kicad_sch")
-    (property "Sheetname" "")
-    (property "exclude_from_bom" "")
+    (property "LCSC" "C160404")
+    (property "Sheetfile" "bmx280-i2c-adapter.kicad_sch")
+    (property "Sheetname" "")
     (property "ki_description" "Generic connector, single row, 01x04, script generated (kicad-library-utils/schlib/autogen/connector/)")
     (property "ki_keywords" "connector")
-    (attr smd exclude_from_pos_files exclude_from_bom)
+    (attr smd)
     (fp_text reference "J2" (at 0 -3.98) (layer "F.SilkS") hide
         (effects (font (size 1 1) (thickness 0.15)))
@@
     (descr "JST SH series connector, SM04B-SRSS-TB (http://www.jst-mfg.com/product/pdf/eng/eSH.pdf), generated with kicad-footprint-generator")
     (tags "connector JST SH top entry")
-    (property "LCSC" "")
-    (property "Sheetfile" "bmx280-i2c-adapter.kicad_sch")
-    (property "Sheetname" "")
-    (property "exclude_from_bom" "")
+    (property "LCSC" "C160404")
+    (property "Sheetfile" "bmx280-i2c-adapter.kicad_sch")
+    (property "Sheetname" "")
     (property "ki_description" "Generic connector, single row, 01x04, script generated (kicad-library-utils/schlib/autogen/connector/)")
     (property "ki_keywords" "connector")
-    (attr smd exclude_from_pos_files exclude_from_bom)
+    (attr smd)
     (fp_text reference "J4" (at 0 -3.98) (layer "F.SilkS") hide
         (effects (font (size 1 1) (thickness 0.15)))
@@
     (descr "JST SH series connector, SM04B-SRSS-TB (http://www.jst-mfg.com/product/pdf/eng/eSH.pdf), generated with kicad-footprint-generator")
     (tags "connector JST SH top entry")
-    (property "LCSC" "")
+    (property "LCSC" "C160404")
     (property "Sheetfile" "bmx280-i2c-adapter.kicad_sch")
     (property "Sheetname" "")
@@
     (descr "JST SH series connector, SM04B-SRSS-TB (http://www.jst-mfg.com/product/pdf/eng/eSH.pdf), generated with kicad-footprint-generator")
     (tags "connector JST SH top entry")
-    (property "LCSC" "")
+    (property "LCSC" "C160404")
     (property "Sheetfile" "bmx280-i2c-adapter.kicad_sch")
     (property "Sheetname" "")
@@
     (effects (font (size 0.8 0.8) (thickness 0.1)) (justify left bottom mirror))
   )
-  (gr_text "Rev: 1.00" (at 119.3 128.25) (layer "B.SilkS")
+  (gr_text "Rev: 1.01" (at 119.3 128.25) (layer "B.SilkS")
     (effects (font (size 1 1) (thickness 0.1)) (justify left bottom mirror))
   )
