File: bmx280-i2c-adapter.kicad/bmx280-i2c-adapter.kicad_sch (KiCad schematic)
At the start: 13 parts, among them J1 Stemma-QT_Qwicc, J2 Stemma-QT_Qwicc, J3 Stemma-QT_Qwicc, J4 Stemma-QT_Qwicc, J5 Grove, J6 Grove, U1 BMx280

Commit message: Rev 1.01: add assembly for Stemma/Qt on top side
Parts:
- J1, J3: LCSC (none) -> C160404
- J2, J4: LCSC (none) -> C160404; now in the parts list
Other:
- note added: "bottom"
- note added: "top"
Changed lines of the file:
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@@
   (title_block
     (title "BMx280 I2C Adapter")
-    (date "2024-08-01")
-    (rev "1.00")
+    (date "2024-08-23")
+    (rev "1.01")
     (company "Bernhard Bablok")
     (comment 1 "https://github.com/bablokb/pcb-bmx280-i2c-adapter")
@@
     (effects (font (size 1.27 1.27)) (justify left bottom))
   )
+  (text "top" (at 140.97 82.55 0)
+    (effects (font (size 1.27 1.27)) (justify left bottom))
+  )
+  (text "bottom" (at 140.97 69.85 0)
+    (effects (font (size 1.27 1.27)) (justify left bottom))
+  )
+  (text "bottom" (at 140.97 95.25 0)
+    (effects (font (size 1.27 1.27)) (justify left bottom))
+  )
+  (text "top" (at 140.97 107.95 0)
+    (effects (font (size 1.27 1.27)) (justify left bottom))
+  )
   (text "0x76" (at 101.6 129.54 0)
     (effects (font (size 1.27 1.27)) (justify left bottom))
@@
   )
   (symbol (lib_id "user:Stemma-QT_Qwicc") (at 133.35 101.6 0) (unit 1)
-    (in_bom no) (on_board yes) (dnp no) (fields_autoplaced)
+    (in_bom yes) (on_board yes) (dnp no) (fields_autoplaced)
     (property "Reference" "J4" (at 140.97 101.6 0)
       (effects (font (size 1.27 1.27)) (justify left))
@@
       (effects (font (size 1.27 1.27)) hide)
     )
-    (property "LCSC" "" (at 133.35 101.6 0)
+    (property "LCSC" "C160404" (at 133.35 101.6 0)
       (effects (font (size 1.27 1.27)) hide)
     )
@@
       (effects (font (size 1.27 1.27)) hide)
     )
-    (property "LCSC" "" (at 133.35 88.9 0)
+    (property "LCSC" "C160404" (at 133.35 88.9 0)
       (effects (font (size 1.27 1.27)) hide)
     )
@@
       (effects (font (size 1.27 1.27)) hide)
     )
-    (property "LCSC" "" (at 133.35 63.5 0)
+    (property "LCSC" "C160404" (at 133.35 63.5 0)
       (effects (font (size 1.27 1.27)) hide)
     )
@@
   )
   (symbol (lib_id "user:Stemma-QT_Qwicc") (at 133.35 76.2 0) (unit 1)
-    (in_bom no) (on_board yes) (dnp no) (fields_autoplaced)
+    (in_bom yes) (on_board yes) (dnp no) (fields_autoplaced)
     (property "Reference" "J2" (at 140.97 76.2 0)
       (effects (font (size 1.27 1.27)) (justify left))
@@
       (effects (font (size 1.27 1.27)) hide)
     )
-    (property "LCSC" "" (at 133.35 76.2 0)
-      (effects (font (size 1.27 1.27)) hide)
-    )
+    (property "LCSC" "C160404" (at 133.35 76.2 0)
+      (effects (font (size 1.27 1.27)) hide)
+    )
